File: circuit/KiCAD_v1.2/nrfburn.kicad_pcb (KiCad board)
At the start: 2 copper layers, 50 x 50 mm, 30 parts, among them IC1 ATMEGA88PA-A, J1 USB, P1 PWR_5V, P3 SWD, U1 AVR-ISP6, U2 MCP1702, U3 LU1_PRG_SPRKFN, U4 LU1_PRG_DNGL, U5 LE1_PRG, U6 DBG_LU1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

Commit message: KiCad schematic and PCB for usable with the new KiCad release (4.0.1)
Parts:
- removed J1: USB, nrfburn:USB_B
- added G***: OSHW-logo_silkscreen-front_12mm, oshw_logo:OSHW-logo_silkscreen-front_12mm, F.Cu at (92.2, 109.2)
- added G***: OSHW-logo_silkscreen-front_12mm, oshw_logo:OSHW-logo_silkscreen-front_12mm, B.Cu at (68.6, 126.2)
- added P2: USB_B, nrfburn:USB_B_loc, F.Cu at (61.6, 104.8)
- moved C1 0.13 mm to (60.6, 123.2)
Connections:
- net +3.3V renamed +3V3
Other:
- board text added: "nrfburn v1.2a (c) 2016 January 21 Ferenc Szili https://github.com/nodep/nrfburn"
- board text removed: "nrfburn v1.2 (c) 2015 August 01 Ferenc Szili https://github.com/nodep/nrfburn"

Commit message: moved HW design to KiCad 8
Parts:
- removed the G*** at (92.2, 109.2)
- removed the G*** at (68.6, 126.2)
- added G***: OSHW-logo_silkscreen-front_12mm, nrfburn:OSHW-logo_silkscreen-front_12mm, F.Cu at (92.1, 109.2)
- added G***: OSHW-logo_silkscreen-back_9mm, nrfburn:OSHW-logo_silkscreen-back_9mm, B.Cu at (93.9, 105.2)
- IC1: value ATMEGA88PA-A -> ATMEGA88PA-AU
- moved U4 1.00 mm to (95.9, 128.0)
Connections:
- IC1 pad 10: (no net) -> unconnected-(IC1-(PCINT22/OC0A/AIN0)PD6-Pad10)
- IC1 pad 11: (no net) -> unconnected-(IC1-(PCINT23/AIN1)PD7-Pad11)
- IC1 pad 19: (no net) -> unconnected-(IC1-ADC6-Pad19)
- IC1 pad 20: (no net) -> unconnected-(IC1-AREF-Pad20)
- IC1 pad 22: (no net) -> unconnected-(IC1-ADC7-Pad22)
- IC1 pad 27: (no net) -> unconnected-(IC1-(PCINT12/SDA/ADC4)PC4-Pad27)
- IC1 pad 28: (no net) -> unconnected-(IC1-(PCINT13/SCL/ADC5)PC5-Pad28)
- IC1 pad 30: (no net) -> unconnected-(IC1-(PCINT16/RXD)PD0-Pad30)
- P2 pad 5: (no net) -> unconnected-(P2-Shield-Pad5)
Other:
- net class Default removed
- board text added: "nrfburn v1.2b (c) 2025 February 16 Ferenc Szili https://github.com/nodep/nrfburn"
- board text removed: "nrfburn v1.2a (c) 2016 January 21 Ferenc Szili https://github.com/nodep/nrfburn"
